File: Hardware/lidar.sch (KiCad schematic (older format))
At the start: 34 parts, among them IC1 A3909GLYTR-T, J1 SENSOR1, J2 SENSOR2, J3 VL53L0X_1, J4 programming, J5 SERVO1, J6 SERVO2, J7 VL53L0X_2, J8 Main conn, J9 Motor, Q1 DMP2100U, SW1 Reset, U1 ATmega328P-AU, U2 MCP25625-x-SS, U3 L7806, U4 L4931, Y1 16MHz resonator, Y2 16MHz resonator

Commit message: Changed digikey link on u3
Parts:
- IC1: symbol A3909GLYTR-T:A3909GLYTR-T -> lidar-rescue:A3909GLYTR-T-A3909GLYTR-T
Changed lines of the file:
@@
 EESchema Schematic File Version 4
 LIBS:lidar-cache
-EELAYER 26 0
+EELAYER 29 0
 EELAYER END
 $Descr A4 11693 8268
@@
 	850  3200 900  3200
 $Comp
-L A3909GLYTR-T:A3909GLYTR-T IC1
+L lidar-rescue:A3909GLYTR-T-A3909GLYTR-T IC1
 U 1 1 5C154A58
 P 9000 950

Commit message: Cleanup, generated schematic
Parts:
- Y1, Y2: value 16MHz resonator -> 16MHz oscillator
Other:
- note added: "ATMEGA328P"
- note added: "Arduino programming\n"
- note added: "BYPASS-CAP"
- note added: "H-BRIDGE"
- note added: "Hall Sensor"
- note added: "I2C pullup\n"
- note added: "MCP25625\n"
- note added: "Main connector"
- note added: "Regulators"
- note added: "Reset and DTR"
- note added: "Servo"
- note added: "VL53L0x"
- moved on the sheet: C1, C2, C3, C5, C6, C7, D1, J1, J2, J3, J4, J5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
